Commit message: fix(urdf): rotate optical frame so X points to old Y position (yaw +pi)

File: src/lerobot_description/urdf/so101_camera_in_hand.xacro (robot description, xacro)
@@ -32,5 +32,5 @@
             <parent link="ee_camera_link"/>
             <child link="ee_camera_optical_link"/>
-            <origin xyz="0 0 0" rpy="-1.5707963 0 -1.5707963"/>
+            <origin xyz="0 0 0" rpy="3.1415927 0 -1.5707963"/>
         </joint>
         <gazebo reference="ee_camera_link">

Commit message: fix: revert optical frame to standard ROS, LookAt=gripperX, PRE_GRASP=Ry(-90)

File: src/lerobot_description/urdf/so101_camera_in_hand.xacro (robot description, xacro)
@@ -32,5 +32,5 @@
             <parent link="ee_camera_link"/>
             <child link="ee_camera_optical_link"/>
-            <origin xyz="0 0 0" rpy="3.1415927 0 -1.5707963"/>
+            <origin xyz="0 0 0" rpy="-1.5707963 0 -1.5707963"/>
         </joint>
         <gazebo reference="ee_camera_link">

Commit message: fix: rotate optical frame blue(Z) to green(Y) pos, update LookAt to -gripperZ

File: src/lerobot_description/urdf/so101_camera_in_hand.xacro (robot description, xacro)
@@ -32,5 +32,5 @@
             <parent link="ee_camera_link"/>
             <child link="ee_camera_optical_link"/>
-            <origin xyz="0 0 0" rpy="-1.5707963 0 -1.5707963"/>
+            <origin xyz="0 0 0" rpy="-1.5707963 0 3.1415927"/>
         </joint>
         <gazebo reference="ee_camera_link">

Commit message: fix: optical Z to old X position, LookAt to -gripperY

File: src/lerobot_description/urdf/so101_camera_in_hand.xacro (robot description, xacro)
@@ -32,5 +32,5 @@
             <parent link="ee_camera_link"/>
             <child link="ee_camera_optical_link"/>
-            <origin xyz="0 0 0" rpy="-1.5707963 0 3.1415927"/>
+            <origin xyz="0 0 0" rpy="3.1415927 0 -1.5707963"/>
         </joint>
         <gazebo reference="ee_camera_link">
