Commit message: fix planning scene

File: src/lerobot_description/urdf/so101_base.xacro (robot description, xacro)
@@ -363,5 +363,5 @@
 		<child link="gripper" />
 		<axis xyz="0 0 1" />
-		<limit effort="10" velocity="10" lower="-2.79253" upper="2.79253" />
+		<limit effort="10" velocity="10" lower="-2.94" upper="2.94" />
 	</joint>
 	<transmission name="5_trans">
@@ -381,5 +381,5 @@
 		<child link="wrist" />
 		<axis xyz="0 0 1" />
-		<limit effort="10" velocity="10" lower="-1.65806" upper="1.65806" />
+		<limit effort="10" velocity="10" lower="-1.80" upper="1.80" />
 	</joint>
 	<transmission name="4_trans">

Commit message: fix: wrist-flip fix for Cartesian approach/sweep + simplified pipeline + physics fixes
- grab_action: force Ry(-90°) downward orientation in _plan_approach
  and _do_push_sweep to prevent 90° wrist flip during Cartesian interp
- grab_action_simple/vlm_bridge_simple: simplified pipeline without
  stage-2 VLM fine localization
- prompts: add GENERIC_STAGE1 prompt for non-strawberry scenarios
- target_box.sdf: enable gravity, increase mass (0.05→5.0) and
  size (0.03→0.05) to fix post-detach flipping
- so101_base.xacro: base_joint Z offset 0.175→0.0
- setup.py: register *_simple entry points

File: src/lerobot_description/urdf/so101_base.xacro (robot description, xacro)
@@ -11,5 +11,5 @@
 		<parent link="world" />
 		<child link="base" />
-		<origin xyz="0 0 0.175" rpy="0 0 0" />
+		<origin xyz="0 0 0.0" rpy="0 0 0" />
 	</joint>
 	<!-- Materials -->
